Commit message: 20th October  finish the ft simulation and urdf

File: baxter_common/rethink_ee_description/urdf/sake_gripper/ezgripper_dual.urdf.xacro (robot description, xacro)
@@ -2,4 +2,6 @@
 <robot name="ezgripper" xmlns:xacro="http://www.ros.org/wiki/xacro">
 <!--macro name="ezgripper" params="*origin"-->
+<xacro:arg name="gazebo" default="false"/>
+<xacro:include filename="$(find baxter_description)/urdf/materials.xacro"/>
 <macro name="ezgripper_dual" params="prefix parent_link *origin">
     <!-- links -->
@@ -10,4 +12,5 @@
           <mesh filename="package://ezgripper_driver/meshes/visual/SAKE_Palm_Dual.stl"/>
         </geometry>
+        <material name="black"/>
       </visual>
       <collision>
@@ -23,5 +26,5 @@
     </link>
     <joint name="${prefix}_ezgripper_connect" type="fixed">
-        <origin rpy="0 0 0" xyz="0.049 0.0 0.1"/>
+        <origin rpy="0 ${-pi/2} 0" xyz="0 0 0"/>
         <parent link="${parent_link}"/>
         <child link="${prefix}_ezgripper_palm_link"/>
@@ -29,4 +32,9 @@
         <limit effort="0" lower="-1.57075" upper="0.25" velocity="3.67"/>
     </joint>
+    <gazebo reference="${prefix}_ezgripper_palm_link">
+      <mu1>0.2</mu1>
+      <mu2>0.2</mu2>
+      <material>Gazebo/White</material>
+    </gazebo>
     <ezgripper_finger prefix="${prefix}" postfix="1" reflect="1" />
     <ezgripper_finger prefix="${prefix}" postfix="2" reflect="1" />
@@ -35,5 +43,5 @@
     <ezgripper_knuckle_trans prefix="${prefix}" postfix="1"/>
     <ezgripper_knuckle_trans prefix="${prefix}" postfix="2"/>
-    <gazebo_knuckle_jsp prefix="${prefix}" />
+   <gazebo_knuckle_jsp prefix="${prefix}" />
 </macro>
 <macro name="ezgripper_finger" params="prefix postfix reflect">
@@ -44,4 +52,5 @@
           <mesh filename="package://ezgripper_driver/meshes/visual/SAKE_Finger.stl"/>
         </geometry>
+         <material name="grey"/>
       </visual>
       <collision>
@@ -56,4 +65,9 @@
       </inertial>
     </link>
+    <gazebo reference="{prefix}_ezgripper_finger_${postfix}">
+      <mu1>0.8</mu1>
+      <mu2>0.8</mu2>
+      <material>Gazebo/Grey</material>
+    </gazebo>
 </macro>
     <!-- joints -->
